File: sowboard/column.kicad_sch (KiCad schematic)
At the start: 9 parts, among them J1 Conn_01x10_MountingPin

Commit message: Improve sowboard layout a bit, switch the data pin to PD2, and work around DRC warnings
Parts:
- removed J1: Conn_01x10_MountingPin, Custom:GCT_FFC2A33-10-T-R_REVA, symbol Connector_Generic_MountingPin:Conn_01x10_MountingPin
- added J1: Conn_01x10_MountingPin, Custom:GCT_FFC2A33-10-T-R_REVA, symbol Connector_Generic:Conn_01x12
Connections:
- net COL: now also J1.5 (Pin_5), J1.6 (Pin_6)
- net R1: now also J1.1 (Pin_1)
- net R2: now also J1.2 (Pin_2)
- net R7: now also J1.9 (Pin_9)
- net R8: now also J1.10 (Pin_10)
- net at D1.2 (A): now also J1.4 (Pin_4)
- net at D3.2 (A): now also J1.8 (Pin_8)
- net at D2.2 (A): now also J1.3 (Pin_3)
- net at D4.2 (A): now also J1.7 (Pin_7)
- no-connect marks 0 -> 2
