File: sowboard/sowboard.kicad_sch (KiCad schematic)
At the start: 8 parts, among them J1 Conn_01x10_MountingPin, U1 ProMicro, U2 PJ-320A, U3 PJ-320A

Commit message: Improve sowboard layout a bit, switch the data pin to PD2, and work around DRC warnings
Parts:
- J1: symbol Connector_Generic_MountingPin:Conn_01x10_MountingPin -> Connector_Generic:Conn_01x12
Connections:
- net at U3.3 (Ring1): now also U1.2 (RX), U1.2B (RX), U2.3 (Ring1); no longer U1.1 (TX)
- net at U3.4 (Ring2): no longer U1.2 (RX)
- net at U2.4 (Ring2): no longer U1.1B (TX)
- removed net GND: J1.MP (MountPin)
- no-connect marks 4 -> 10
Changed lines of the file:
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@@
 (kicad_sch (version 20230121) (generator eeschema)
   (paper "A4")
+  (junction (at 205.74 85.09) (diameter 0) (color 0 0 0 0)
+  )
+  (junction (at 170.18 52.07) (diameter 0) (color 0 0 0 0)
+  )
   (junction (at 208.28 52.07) (diameter 0) (color 0 0 0 0)
   )
+  (no_connect (at 205.74 87.63))
+  (no_connect (at 110.49 143.51))
   (no_connect (at 205.74 54.61))
+  (no_connect (at 193.04 24.13))
+  (no_connect (at 189.23 106.68))
+  (no_connect (at 170.18 49.53))
   (no_connect (at 170.18 57.15))
   (no_connect (at 205.74 49.53))
+  (no_connect (at 110.49 140.97))
   (no_connect (at 170.18 54.61))
   (wire (pts (xy 194.31 102.87) (xy 194.31 91.44))
@@
     (stroke (width 0) (type default))
   )
+  (wire (pts (xy 187.96 85.09) (xy 205.74 85.09))
+    (stroke (width 0) (type default))
+  )
   (wire (pts (xy 208.28 52.07) (xy 205.74 52.07))
     (stroke (width 0) (type default))
@@
     (stroke (width 0) (type default))
   )
-  (wire (pts (xy 193.04 24.13) (xy 201.93 24.13))
-    (stroke (width 0) (type default))
-  )
   (wire (pts (xy 205.74 59.69) (xy 208.28 59.69))
     (stroke (width 0) (type default))
@@
     (stroke (width 0) (type default))
   )
-  (wire (pts (xy 189.23 106.68) (xy 205.74 106.68))
-    (stroke (width 0) (type default))
-  )
   (wire (pts (xy 193.04 31.75) (xy 208.28 31.75))
     (stroke (width 0) (type default))
@@
     (stroke (width 0) (type default))
   )
+  (wire (pts (xy 207.01 110.49) (xy 189.23 110.49))
+    (stroke (width 0) (type default))
+  )
   (wire (pts (xy 189.23 102.87) (xy 194.31 102.87))
     (stroke (width 0) (type default))
   )
-  (wire (pts (xy 207.01 110.49) (xy 207.01 85.09))
-    (stroke (width 0) (type default))
-  )
   (wire (pts (xy 139.7 135.89) (xy 139.7 154.94))
     (stroke (width 0) (type default))
@@
     (stroke (width 0) (type default))
   )
-  (wire (pts (xy 167.64 40.64) (xy 167.64 52.07))
-    (stroke (width 0) (type default))
-  )
   (wire (pts (xy 167.64 80.01) (xy 170.18 80.01))
     (stroke (width 0) (type default))
   )
-  (wire (pts (xy 189.23 110.49) (xy 207.01 110.49))
-    (stroke (width 0) (type default))
-  )
-  (wire (pts (xy 201.93 40.64) (xy 167.64 40.64))
+  (wire (pts (xy 207.01 85.09) (xy 205.74 85.09))
     (stroke (width 0) (type default))
   )
@@
     (stroke (width 0) (type default))
   )
-  (wire (pts (xy 201.93 24.13) (xy 201.93 40.64))
-    (stroke (width 0) (type default))
-  )
   (wire (pts (xy 208.28 59.69) (xy 208.28 52.07))
     (stroke (width 0) (type default))
   )
+  (wire (pts (xy 170.18 52.07) (xy 187.96 52.07))
+    (stroke (width 0) (type default))
+  )
   (wire (pts (xy 208.28 31.75) (xy 208.28 52.07))
     (stroke (width 0) (type default))
   )
-  (wire (pts (xy 167.64 52.07) (xy 170.18 52.07))
+  (wire (pts (xy 187.96 52.07) (xy 187.96 85.09))
     (stroke (width 0) (type default))
   )
@@
     (stroke (width 0) (type default))
   )
-  (wire (pts (xy 204.47 41.91) (xy 170.18 41.91))
+  (wire (pts (xy 204.47 41.91) (xy 166.37 41.91))
     (stroke (width 0) (type default))
   )
@@
     (stroke (width 0) (type default))
   )
-  (wire (pts (xy 170.18 41.91) (xy 170.18 49.53))
-    (stroke (width 0) (type default))
-  )
-  (wire (pts (xy 205.74 87.63) (xy 205.74 106.68))
-    (stroke (width 0) (type default))
-  )
-  (wire (pts (xy 207.01 85.09) (xy 205.74 85.09))
+  (wire (pts (xy 166.37 41.91) (xy 166.37 52.07))
+    (stroke (width 0) (type default))
+  )
+  (wire (pts (xy 207.01 85.09) (xy 207.01 110.49))
+    (stroke (width 0) (type default))
+  )
+  (wire (pts (xy 166.37 52.07) (xy 170.18 52.07))
     (stroke (width 0) (type default))
   )
@@
     )
   )
-  (symbol (lib_id "power:GND") (at 105.41 143.51 0) (unit 1)
-    (in_bom yes) (on_board yes) (dnp no) (fields_autoplaced)
-    (property "Reference" "#PWR04" (at 105.41 149.86 0)
-      (effects (font (size 1.27 1.27)) hide)
-    )
-    (property "Value" "GND" (at 105.41 148.59 0)
-      (effects (font (size 1.27 1.27)) hide)
-    )
-    (property "Footprint" "" (at 105.41 143.51 0)
-      (effects (font (size 1.27 1.27)) hide)
-    )
-    (property "Datasheet" "" (at 105.41 143.51 0)
-      (effects (font (size 1.27 1.27)) hide)
-    )
-    (pin "1")
-    (instances
-      (project "sowboard"
-        (path "/4cf5c873-f5e9-4261-911c-886f387fb0f3"
-          (reference "#PWR04") (unit 1)
-        )
-      )
-    )
-  )
   (symbol (lib_id "Diode:1N4148W") (at 114.3 133.35 180) (unit 1)
     (in_bom yes) (on_board yes) (dnp no) (fields_autoplaced)
@@
     )
   )
-  (symbol (lib_id "Connector_Generic_MountingPin:Conn_01x10_MountingPin") (at 105.41 125.73 0) (mirror y) (unit 1)
+  (symbol (lib_id "Connector_Generic:Conn_01x12") (at 105.41 128.27 0) (mirror y) (unit 1)
     (in_bom yes) (on_board yes) (dnp no)
-    (property "Reference" "J1" (at 102.87 126.7206 0)
+    (property "Reference" "J1" (at 102.87 129.2606 0)
       (effects (font (size 1.27 1.27)) (justify left))
     )
-    (property "Value" "Conn_01x10_MountingPin" (at 102.87 129.2606 0)
+    (property "Value" "Conn_01x10_MountingPin" (at 102.87 131.8006 0)
       (effects (font (size 1.27 1.27)) (justify left))
     )
-    (property "Footprint" "Custom:GCT_FFC2A33-10-T-R_REVA" (at 105.41 125.73 0)
-      (effects (font (size 1.27 1.27)) hide)
-    )
-    (property "Datasheet" "~" (at 105.41 125.73 0)
+    (property "Footprint" "Custom:GCT_FFC2A33-10-T-R_REVA" (at 105.41 128.27 0)
+      (effects (font (size 1.27 1.27)) hide)
+    )
+    (property "Datasheet" "~" (at 105.41 128.27 0)
       (effects (font (size 1.27 1.27)) hide)
     )
     (pin "1")
     (pin "10")
+    (pin "S1")
+    (pin "S2")
     (pin "2")
     (pin "3")
@@
     (pin "8")
     (pin "9")
-    (pin "MP")
     (instances
       (project "sowboard"
